File: projects/LED Analog Watch/led_analog_watch_mvmt_v1_2.brd (EAGLE design)
At the start: 35.6 x 35.6 mm, 47 parts, among them IC1 ATMEGA644M, IC2 FT232RQ, U2 MCP73831, Y1 32kHz

Commit message: Minor adjustments to schematic and docs
Parts:
- renumbered IC1 to MCU, IC2 to USB_SERIAL, JP1 to µUSB, U$1 to RTC, U2 to USB_CHARGER
