File: projects/Digital Clock/Digital Clock v2.brd (EAGLE design)
At the start: 82.5 x 101 mm, 43 parts, among them U1 FT232RL-BASICSSOP

Commit message: Many minor revisions to Digital Clock v2
Parts:
- added FRAME1: FRAME-LETTERNO_PACKAGE, jcole:DUMMY
- REG_3V3: value LD33V -> LT1521CST-3.3; device SparkFun:78XXL -> jcole:SOT223
- REG_5V0: value L7805 -> LT1521CST-5; device SparkFun:78XXL -> jcole:SOT223
Connections:
- removed net N$3: PWR.3
- net GND: now also REG_3V3.2, REG_3V3.TAB, REG_5V0.2, REG_5V0.TAB; no longer REG_3V3.GND, REG_5V0.GND
- net LCD_MISO: now also LCD_ICSP_TC.1
- net LCD_MOSI: no longer LCD_ICSP_TC.1
- net VCC_3V3: now also REG_3V3.3; no longer REG_3V3.OUT
- net VCC_5V0: now also REG_3V3.1, REG_5V0.3; no longer REG_3V3.IN, REG_5V0.OUT
- net VIN_SW: now also REG_5V0.1; no longer REG_5V0.IN
Routing:
- net GND: track 364.9 -> 0.00 mm, vias 1 -> 0
- net VCC_5V0: track 216.8 -> 0.00 mm, vias 1 -> 0
- net VCC_3V3: track 167.9 -> 0.00 mm, vias 5 -> 0
- net LCD_TXD: track 125.9 -> 0.00 mm, vias 1 -> 0
- net LCD_SCK: track 114.3 -> 0.00 mm, vias 2 -> 0
- net LCD_RST: track 107.9 -> 0.00 mm, vias 2 -> 0
- net LCD_RXD: track 102.1 -> 0.00 mm, vias 1 -> 0
- net LCD_MOSI: track 99.1 -> 0.00 mm, vias 2 -> 0
- net SDA: track 98.7 -> 0.00 mm, vias 1 -> 0
- net SCL: track 91.4 -> 0.00 mm, vias 1 -> 0
- net N$7: track 75.6 -> 0.00 mm, vias 3 -> 0
- net VIN: track 62.1 -> 0.00 mm
- net N$17: track 59.0 -> 0.00 mm, vias 5 -> 0
- net LED_RXD: track 58.2 -> 0.00 mm, vias 1 -> 0
- net GPS_TXD: track 54.7 -> 0.00 mm, vias 3 -> 0
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Other:
- board text added: "3V3"
- board text added: "5V0"
